File: Telegraph.kicad_pcb (KiCad board)
At the start: 2 copper layers, 99.7 x 66 mm, 100 parts, among them CON1 BARREL_JACK, J1 Raspberry_Pi_2_3, P1 SPK, P2 KEY, P3 STEPPER, P4 MAGNETS, P5 FTDI-DEVICE, Q1 STU60N3LH5, Q2 STU60N3LH5, SW1 SW_Push

Commit message: Improve values for speaker
The previous resistor values were more conservative, based on another
speaker.  Testing with the actual speaker, whose type number was also
addd to the schematic, suggests smaller resistor values will work
better.
Parts:
- R2: value 47R -> 12R
- RV1: value 1K -> 100R
- SP1: value SPEAKER -> CVS-1508
Changed lines of the file:
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@@
     (links 137)
     (no_connects 0)
-    (area 40.410001 41.75 160.020001 119.380001)
+    (area 53.264999 50.724999 153.110001 116.915001)
     (thickness 1.6)
     (drawings 13)
@@
       (effects (font (size 1 1) (thickness 0.15)))
     )
-    (fp_text value 1K (at 5 3.65 180) (layer F.Fab)
+    (fp_text value 100R (at 5 3.65 180) (layer F.Fab)
       (effects (font (size 1 1) (thickness 0.15)))
     )
@@
       (effects (font (size 1 1) (thickness 0.15)))
     )
-    (fp_text value SPEAKER (at 3.81 8.89 90) (layer F.Fab)
+    (fp_text value CVS-1508 (at 3.81 8.89 90) (layer F.Fab)
       (effects (font (size 1 1) (thickness 0.15)))
     )
@@
       (effects (font (size 1 1) (thickness 0.15)))
     )
-    (fp_text value 47R (at 5.08 2.31) (layer F.Fab)
-      (effects (font (size 1 1) (thickness 0.15)))
-    )
+    (fp_text value 12R (at 5.08 2.31) (layer F.Fab)
+      (effects (font (size 1 1) (thickness 0.15)))
+    )

Commit message: Convert to KiCad 5
There might be other changes too, I did not commit this right away...
Routing:
- net (no net): track 0.00 -> 1.27 mm
